File: main.kicad_sch (KiCad schematic)
At the start: 84 parts, among them J1 USB_C_Receptacle, J2 Bus_M.2_Socket_M, U2 SPI_SOIC-8, U3 SPI_DFN-8, Y1 25MHz

Commit message: added no connects, refclocks and perst for -PDX
Connections:
- net REFCLK+: no longer U1.AA8 (REFCLKP0)
- net REFCLK-: no longer U1.Y8 (REFCLKN0)
- net REFCLK2+: now reaches U1.AA10 (NC/REFCLKP2)
- net REFCLK1+: now reaches U1.AA11 (NC/REFCLKP1)
- net REFCLK3+: now reaches U1.AA7 (NC/REFCLKP3)
- net PERST3#: now reaches U1.D21 (NC/PERST3#)
- net PERST2#: now reaches U1.E21 (NC/PERST2#)
- net PERST1#: now reaches U1.F21 (NC/PERST1#)
- net REFCLK2-: now reaches U1.Y10 (NC/REFCLKN2)
- net REFCLK1-: now reaches U1.Y11 (NC/REFCLKN1)
- net REFCLK3-: now reaches U1.Y7 (NC/REFCLKN3)
- new net REFCLK0+: U1.AA8 (REFCLKP0)
- new net REFCLK0-: U1.Y8 (REFCLKN0)
- no-connect marks 2 -> 34
